Commit message: basic implementation of the hardware interface

File: config/hardware_interface.ros2_control.xacro (robot description, xacro)
@@ -1,10 +1,23 @@
 <?xml version="1.0"?>
 <robot xmlns:xacro="http://www.ros.org.wiki/xacro">
-    <xacrop:property name="pi" value="3.145"/>
-    <ros2_control name="quaro_hardware_interface" type="system">
+    <ros2_control name="quaro_legs_hardware_interface" type="system">
         <hardware>
             <plugin>quaro_hardware_interface/QuaroSystem</plugin>
         </hardware>
-        <joint name="joint_0">
+        <joint name="hip_0">
+            <command_interface name="position">
+                <param name="min">${-135/180*pi}</param>
+                <param name="max">${135/180*pi}</param>
+            </command_interface>
+            <state_interface name="position"/>
+        </joint>
+        <joint name="knee_0">
+            <command_interface name="position">
+                <param name="min">${-135/180*pi}</param>
+                <param name="max">${135/180*pi}</param>
+            </command_interface>
+            <state_interface name="position"/>
+        </joint>
+        <joint name="ankle_0">
             <command_interface name="position">
                 <param name="min">${-135/180*pi}</param>
