Commit message: correctly include the macro, correct interface name for the battery and correct entries for the joints

File: ros2_control/hardware_interface.ros2_control.xacro (robot description, xacro)
@@ -1,6 +1,6 @@
 <?xml version="1.0"?>
-<xacro:include filename='$(find quaro_hardware_interface)/ros2_control/lx224hw_inferface.ros2_control.xacro'/>
 <robot xmlns:xacro="http://www.ros.org.wiki/xacro">
-    <xacro:macro name="quaro_ros2_control" params="name">
+    <xacro:include filename='$(find quaro_hardware_interface)/ros2_control/lx224hv_interface.ros2_control.xacro'/>
+    <xacro:macro name="quaro_ros2_control">
         <ros2_control name="quaro_legs_hardware_interface" type="system">
             <hardware>
@@ -28,5 +28,5 @@
             </sensor>
             <sensor name="battery">
-                <state_interface name="voltage"/>
+                <state_interface name="battery_voltage"/>
             </sensor>
         </ros2_control>

File: ros2_control/lx224hv_interface.ros2_control.xacro (robot description, xacro)
@@ -4,8 +4,8 @@
         <joint name="${name}">
             <command_interface name="position">
-                <param name="min_angle">${-120/180*pi}</param>
-                <param name="min_input">0</param>
-                <param name="max_angle">${120/180*pi}</param>
-                <param name="max_input">1000</param>
+                <param name="min">${-120/180*pi}</param>
+                <!-- <param name="min_input">0</param> -->
+                <param name="max">${120/180*pi}</param>
+                <!-- <param name="max_input">1000</param> -->
             </command_interface>
             <state_interface name="position"/>
